File: pic_programmer.kicad_pcb (KiCad board)
At the start: 2 copper layers, 160 x 99.1 mm, 63 parts, among them J1 DB9-FEMAL, P1 CONN_2, P101 CONN_1, P102 CONN_1, P103 CONN_1, P104 CONN_1, P105 CONN_1, P106 CONN_1, P2 SUPP28, P3 SUPP40, Q1 BC237, Q2 BC307, Q3 BC307, U1 24Cxx, U2 74HC125, U3 7805, U4 LT1373, U5 PIC_18_PINS, U6 PIC_8_PINS

Commit message: Add PDF output
Other:
- board text added: "This text is on User.Drawings layer"
Changed lines of the file:
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@@
     (effects (font (size 2.032 1.524) (thickness 0.3048)) (justify mirror))
+  )
+  (gr_text "This text is on User.Drawings layer" (at 222.25 152.4) (layer "Dwgs.User")
+    (effects (font (size 3 3) (thickness 0.15)))
   )
   (segment (start 85.09 123.19) (end 86.36 124.46) (width 0.5) (layer "B.Cu") (net 1))
