File: pic_programmer.kicad_sch (KiCad schematic)
At the start: 56 parts, among them J1 DB9-FEMAL, P1 CONN_2, P101 CONN_1, P102 CONN_1, P103 CONN_1, P104 CONN_1, P105 CONN_1, P106 CONN_1, Q1 BC237, Q2 BC307, Q3 BC307, U2 74HC125, U3 7805, U4 LT1373

Commit message: Make C4 DNP
Parts:
- C4: BOM (none) -> DNP
Changed lines of the file:
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@@
       (effects (font (size 1.524 1.524)) hide)
+    )
+    (property "BOM" "DNP" (id 4) (at 224.79 160.02 90)
+      (effects (font (size 1.27 1.27)) hide)
     )
     (pin "1")

Commit message: Add optional variable
Other:
- note added: "${OPTIONAL_VARIABLE}"
Changed lines of the file:
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@@
     (effects (font (size 1.524 1.524)) (justify left bottom))
+  )
+  (text "${OPTIONAL_VARIABLE}" (at 179.07 172.72 0)
+    (effects (font (size 2.54 2.54)) (justify left bottom))
   )
   (text "TXD" (at 46.99 91.44 0)
